Commit message: Add inertial, anche ad URDF braccio

File: ws_ur5e_ballpool/src/left_arm_description/urdf/left_arm.urdf.xacro (robot description, xacro)
@@ -74,4 +74,11 @@
             </geometry>
         </collision>
+        <inertial>
+            <origin xyz="-0.001639 -0.002797 0.050174" rpy="0 0 0" />
+            <mass value="0.411613" />
+            <inertia ixx="0.0007612662" ixy="0.0000017135" ixz="0.0000371988"
+                      iyy="0.0007890698" iyz="-0.0000754243"
+                      izz="0.0003099597" />
+        </inertial>
     </link>
     <!-- fixed joint: flangia -> holder -->

Commit message: Separata mazza da holder

File: ws_ur5e_ballpool/src/left_arm_description/urdf/left_arm.urdf.xacro (robot description, xacro)
@@ -9,5 +9,5 @@
     <xacro:arg name="tf_prefix_left" default="left_" />
     <!-- LETTURA PARAMETRI DELL'UR5e DA CONFIG FILES -->
-    <!-- da ur_description (generici UR)-->
+    <!-- da ur_description, pacchetto ROS (generici UR5e)-->
     <xacro:arg name="joint_limit_params" default="$(find ur_description)/config/$(arg ur_type)/joint_limits.yaml"/>
     <xacro:arg name="physical_params" default="$(find ur_description)/config/$(arg ur_type)/physical_parameters.yaml"/>
@@ -38,54 +38,4 @@
         </collision>
     </link>
-    <!-- left arm -->
-    <xacro:ur_robot
-        name="ur5e"
-        tf_prefix="$(arg tf_prefix_left)"
-        parent="world"
-        joint_limits_parameters_file="$(arg joint_limit_params)"
-        kinematics_parameters_file="$(arg kinematics_params)"
-        physical_parameters_file="$(arg physical_params)"
-        visual_parameters_file="$(arg visual_params)"
-        safety_limits="$(arg safety_limits)"
-        safety_pos_margin="$(arg safety_pos_margin)"
-        safety_k_position="$(arg safety_k_position)"
-        >
-        <origin xyz="-0.188189 0.13575 0.556631" rpy="${3*pi/4} 0 ${-pi/2}" />
-    </xacro:ur_robot>
-    <!-- gripper/holder link -->
-    <link name="$(arg tf_prefix_left)holder_link">
-        <visual>
-            <origin xyz="0 0 0" rpy="0 0 0" />
-            <geometry>
-                <!-- <mesh filename="package://left_arm_description/meshes/holder/holder.stl" scale="0.001 0.001 0.001"/> -->
-                <!-- <mesh filename="package://left_arm_description/meshes/holder/holder_with_full_rod.stl" scale="0.001 0.001 0.001"/> -->
-                <mesh filename="package://left_arm_description/meshes/holder/holder_with_cut_rod.obj" scale="0.001 0.001 0.001"/>
-            </geometry>
-            <!-- <material name="Grey">     decommenta se non hai usato un obj con mtl file per il colore del mesh (es stl)
-                <color rgba="0.5 0.5 0.5 1.0" />
-            </material> -->
-        </visual>
-        <collision>
-            <origin xyz="0 0 0" rpy="0 0 0" />
-            <geometry>
-                <!-- <mesh filename="package://left_arm_description/meshes/holder/holder.stl" scale="0.001 0.001 0.001"/> -->
-                <!-- <mesh filename="package://left_arm_description/meshes/holder/holder_with_full_rod.stl" scale="0.001 0.001 0.001"/> -->
-                <mesh filename="package://left_arm_description/meshes/holder/holder_with_cut_rod.obj" scale="0.001 0.001 0.001"/>
-            </geometry>
-        </collision>
-        <inertial>
-            <origin xyz="-0.001639 -0.002797 0.050174" rpy="0 0 0" />
-            <mass value="0.411613" />
-            <inertia ixx="0.0007612662" ixy="0.0000017135" ixz="0.0000371988"
-                      iyy="0.0007890698" iyz="-0.0000754243"
-                      izz="0.0003099597" />
-        </inertial>
-    </link>
-    <!-- fixed joint: flangia -> holder -->
-    <joint name="$(arg tf_prefix_left)tool0_holder_joint" type="fixed">
-        <parent link="$(arg tf_prefix_left)tool0" />
-        <child link="$(arg tf_prefix_left)holder_link" />
-        <origin xyz="0 0 0" rpy="0 0 0" />
-    </joint>
     <!-- muro dietro la scrivania -->
     <link name="wall_link">
@@ -111,3 +61,78 @@
         <origin xyz="0 0 0" rpy="0 0 0" />
     </joint>
+    <!-- left arm -->
+    <xacro:ur_robot
+        name="ur5e"
+        tf_prefix="$(arg tf_prefix_left)"
+        parent="world"
+        joint_limits_parameters_file="$(arg joint_limit_params)"
+        kinematics_parameters_file="$(arg kinematics_params)"
+        physical_parameters_file="$(arg physical_params)"
+        visual_parameters_file="$(arg visual_params)"
+        safety_limits="$(arg safety_limits)"
+        safety_pos_margin="$(arg safety_pos_margin)"
+        safety_k_position="$(arg safety_k_position)"
+        >
+        <origin xyz="-0.188189 0.13575 0.556631" rpy="${3*pi/4} 0 ${-pi/2}" />
+    </xacro:ur_robot>
+    <!-- 1. LINK: HOLDER (CAD) -->
+    <link name="$(arg tf_prefix_left)holder_link">
+        <visual>
+            <origin xyz="0 0 0" rpy="0 0 0" />
+            <geometry>
+                <mesh filename="package://left_arm_description/meshes/holder/holder.obj" scale="0.001 0.001 0.001"/>
+            </geometry>
+        </visual>
+        <collision>
+            <origin xyz="0 0 0" rpy="0 0 0" />
+            <geometry>
+                <mesh filename="package://left_arm_description/meshes/holder/holder.obj" scale="0.001 0.001 0.001"/>
+            </geometry>
+        </collision>
+        <inertial>
+            <!-- Centro di massa dell'Holder in metri -->
+            <origin xyz="-0.000040 -0.002910 0.047880" rpy="0 0 0" />
+            <mass value="0.395622" />
+            <inertia ixx="0.0007072540" ixy="-0.0000001274" ixz="-0.0000001817"
+                      iyy="0.0006607535" iyz="-0.0000727837"
+                      izz="0.0002350857" />
+        </inertial>
+    </link>
+    <!-- FIXED JOINT: FLANGIA (tool0) -> HOLDER -->
+    <joint name="$(arg tf_prefix_left)tool0_holder_joint" type="fixed">
+        <parent link="$(arg tf_prefix_left)tool0" />
+        <child link="$(arg tf_prefix_left)holder_link" />
+        <origin xyz="0 0 0" rpy="0 0 0" />
+    </joint>
+    <!-- 2. LINK: CUT ROD -->
+    <link name="$(arg tf_prefix_left)cut_rod_link">
+        <visual>
+            <origin xyz="0 0 0" rpy="0 0 0" />
+            <geometry>
+                <!-- Modifica il percorso se la mesh della rod è in un file separato -->
+                <mesh filename="package://left_arm_description/meshes/holder/cut_rod.obj" scale="0.001 0.001 0.001"/>
+            </geometry>
+        </visual>
+        <collision>
+            <origin xyz="0 0 0" rpy="0 0 0" />
+            <geometry>
+                <mesh filename="package://left_arm_description/meshes/holder/cut_rod.obj" scale="0.001 0.001 0.001"/>
+            </geometry>
+        </collision>
+        <inertial>
+            <!-- Centro di massa della Cut Rod in metri -->
+            <origin xyz="-0.041200 0.000000 0.106920" rpy="0 0 0" />
+            <mass value="0.015991" />
+            <inertia ixx="0.0000003074" ixy="0.0000000000" ixz="0.0000000307"
+                      iyy="0.0000487030" iyz="0.0000000000"
+                      izz="0.0000487052" />
+        </inertial>
+    </link>
+    <!-- FIXED JOINT: HOLDER -> CUT ROD -->
+    <joint name="$(arg tf_prefix_left)holder_cut_rod_joint" type="fixed">
+        <parent link="$(arg tf_prefix_left)holder_link" />
+        <child link="$(arg tf_prefix_left)cut_rod_link" />
+        <!-- Se le mesh condividono lo stesso sistema di riferimento zero del CAD, l'origine è 0 0 0 -->
+        <origin xyz="0 0 0" rpy="0 0 0" />
+    </joint>
 </robot>

Commit message: Aggiornato MuJoco environment e Xacro con nuovo end-effector

File: ws_ur5e_ballpool/src/left_arm_description/urdf/left_arm.urdf.xacro (robot description, xacro)
@@ -92,9 +92,9 @@
         <inertial>
             <!-- Centro di massa dell'Holder in metri -->
-            <origin xyz="-0.000040 -0.002910 0.047880" rpy="0 0 0" />
-            <mass value="0.395622" />
-            <inertia ixx="0.0007072540" ixy="-0.0000001274" ixz="-0.0000001817"
-                      iyy="0.0006607535" iyz="-0.0000727837"
-                      izz="0.0002350857" />
+            <origin xyz="-0.000020 -0.000000 0.034870" rpy="0 0 0" />
+            <mass value="0.190087" />
+            <inertia ixx="0.0002082050" ixy="-0.0000000001" ixz="0.0000002035"
+                     iyy="0.0002077921" iyz="-0.0000000002"
+                     izz="0.0000715583" />
         </inertial>
     </link>
@@ -110,5 +110,4 @@
             <origin xyz="0 0 0" rpy="0 0 0" />
             <geometry>
-                <!-- Modifica il percorso se la mesh della rod è in un file separato -->
                 <mesh filename="package://left_arm_description/meshes/holder/cut_rod.obj" scale="0.001 0.001 0.001"/>
             </geometry>
@@ -122,9 +121,9 @@
         <inertial>
             <!-- Centro di massa della Cut Rod in metri -->
-            <origin xyz="-0.041200 0.000000 0.106920" rpy="0 0 0" />
-            <mass value="0.015991" />
-            <inertia ixx="0.0000003074" ixy="0.0000000000" ixz="0.0000000307"
-                      iyy="0.0000487030" iyz="0.0000000000"
-                      izz="0.0000487052" />
+          <origin xyz="-0.029300 0.000000 0.080990" rpy="0 0 0" />
+          <mass value="0.012517" />
+          <inertia ixx="0.0000002222" ixy="0.0000000000" ixz="0.0000000000"
+                   iyy="0.0000262241" iyz="0.0000000000"
+                   izz="0.0000262242" />
         </inertial>
     </link>

Commit message: Aggiunto tip joint virtuale al robot

File: ws_ur5e_ballpool/src/left_arm_description/urdf/left_arm.urdf.xacro (robot description, xacro)
@@ -135,3 +135,16 @@
         <origin xyz="0 0 0" rpy="0 0 0" />
     </joint>
+    <!-- ========================================== -->
+    <!-- 3. LINK VIRTUALE: ROD TIP (TCP Punta Asta) -->
+    <!-- ========================================== -->
+    <link name="$(arg tf_prefix_left)rod_tip_virtual_link" />
+    <!-- FIXED JOINT: CUT ROD -> ROD TIP VIRTUAL -->
+    <joint name="$(arg tf_prefix_left)cut_rod_tip_joint" type="fixed">
+        <parent link="$(arg tf_prefix_left)cut_rod_link" />
+        <child link="$(arg tf_prefix_left)rod_tip_virtual_link" />
+        <!-- Traslazione in metri: x = -120mm, z = 81mm -->
+        <!-- Rotazione: pitch di -90 gradi (-pi/2) per allineare asse Z su asse -X -->
+        <origin xyz="-0.120 0 0.081" rpy="0 ${-pi/2} 0" />
+    </joint>
+    <!-- NOTA: ANDRÀ TARATO REALISTIACAMENTE CON IL METODO DEL PIVOT!! -->
 </robot>

Commit message: shot execution

File: ws_ur5e_ballpool/src/left_arm_description/urdf/left_arm.urdf.xacro (robot description, xacro)
@@ -145,5 +145,5 @@
         <!-- Traslazione in metri: x = -120mm, z = 81mm -->
         <!-- Rotazione: pitch di -90 gradi (-pi/2) per allineare asse Z su asse -X -->
-        <origin xyz="-0.120 0 0.081" rpy="0 ${-pi/2} 0" />
+        <origin xyz="-0.118 0 0.081" rpy="0 ${-pi/2} 0" />
     </joint>
     <!-- NOTA: ANDRÀ TARATO REALISTIACAMENTE CON IL METODO DEL PIVOT!! -->

File: ws_ur5e_ballpool/src/moveit_config/config/left_arm_ur5e.ros2_control.xacro (robot description, xacro)
@@ -7,8 +7,8 @@
                 <!-- Qui si ha una lista di plugin: decommentare quello che si vuole usare, e commentare gli altri. -->
                 <!-- PLUGIN PER MUJOCO -->
-                <!-- <plugin>mujoco_ros2_control/MujocoSystemInterface</plugin>
-                <param name="mujoco_model">$(find moveit_config)/config/mujoco_bridge/complete_scene.xml</param> -->
+                <plugin>mujoco_ros2_control/MujocoSystemInterface</plugin>
+                <param name="mujoco_model">$(find moveit_config)/config/mujoco_bridge/complete_scene.xml</param>
                 <!-- PLUGIN PER SOLO RVIZ SIMULATO -->
-                <plugin>mock_components/GenericSystem</plugin>
+                <!-- <plugin>mock_components/GenericSystem</plugin> -->
                 <!-- PLUGIN PER HARDWARE REALE -->
                 <!-- ... TODO -->
