Commit message: removed left_

File: ws_ur5e_ballpool/src/arm_description/urdf/arm.urdf.xacro (robot description, xacro)
@@ -1,4 +1,4 @@
 <?xml version="1.0"?>
-<robot name="left_arm_ur5e" xmlns:xacro="http://ros.org/wiki/xacro">
+<robot name="arm_ur5e" xmlns:xacro="http://ros.org/wiki/xacro">
     <!-- robot name parameter -->
     <xacro:arg name="name" default="ur5e"/>
@@ -7,5 +7,5 @@
     <!-- ROBOT XACRO PARAMETERS-->
     <xacro:arg name="ur_type" default="ur5e"/>
-    <xacro:arg name="tf_prefix_left" default="left_" />
+    <xacro:arg name="tf_prefix_left" default="" />
     <!-- LETTURA PARAMETRI DELL'UR5e DA CONFIG FILES -->
     <!-- da ur_description, pacchetto ROS (generici UR5e)-->
@@ -14,5 +14,5 @@
     <xacro:arg name="visual_params" default="$(find ur_description)/config/$(arg ur_type)/visual_parameters.yaml"/>
     <!-- da calibrazione su nostro braccio -->
-    <xacro:arg name="kinematics_params" default="$(find left_arm_description)/config/uclv_left_ur5e_kinematics.yaml"/>
+    <xacro:arg name="kinematics_params" default="$(find arm_description)/config/uclv_right_ur5e_kinematics.yaml"/>
     <!-- safety parameters (ininfluenti in visualizzazione)-->
     <xacro:arg name="safety_limits" default="true"/>
@@ -25,5 +25,5 @@
             <origin xyz="0 0 0" rpy="0 0 0" />
             <geometry>
-                <mesh filename="package://left_arm_description/meshes/vention/visual/myvention_visual.stl" scale="0.001 0.001 0.001"/>
+                <mesh filename="package://arm_description/meshes/vention/visual/myvention_visual.stl" scale="0.001 0.001 0.001"/>
             </geometry>
             <material name="Blue">
@@ -34,5 +34,5 @@
             <origin xyz="0 0 0" rpy="0 0 0" />
             <geometry>
-                <mesh filename="package://left_arm_description/meshes/vention/collision/myvention_collision.stl" scale="0.001 0.001 0.001"/>
+                <mesh filename="package://arm_description/meshes/vention/collision/myvention_collision.stl" scale="0.001 0.001 0.001"/>
             </geometry>
         </collision>
@@ -81,5 +81,5 @@
             <origin xyz="0 0 0" rpy="0 0 0" />
             <geometry>
-                <mesh filename="package://left_arm_description/meshes/holder/holder.obj" scale="0.001 0.001 0.001"/>
+                <mesh filename="package://arm_description/meshes/holder/holder.obj" scale="0.001 0.001 0.001"/>
             </geometry>
         </visual>
@@ -87,5 +87,5 @@
             <origin xyz="0 0 0" rpy="0 0 0" />
             <geometry>
-                <mesh filename="package://left_arm_description/meshes/holder/holder.obj" scale="0.001 0.001 0.001"/>
+                <mesh filename="package://arm_description/meshes/holder/holder.obj" scale="0.001 0.001 0.001"/>
             </geometry>
         </collision>
@@ -110,5 +110,5 @@
             <origin xyz="0 0 0" rpy="0 0 0" />
             <geometry>
-                <mesh filename="package://left_arm_description/meshes/holder/cut_rod.obj" scale="0.001 0.001 0.001"/>
+                <mesh filename="package://arm_description/meshes/holder/cut_rod.obj" scale="0.001 0.001 0.001"/>
             </geometry>
         </visual>
@@ -116,5 +116,5 @@
             <origin xyz="0 0 0" rpy="0 0 0" />
             <geometry>
-                <mesh filename="package://left_arm_description/meshes/holder/cut_rod.obj" scale="0.001 0.001 0.001"/>
+                <mesh filename="package://arm_description/meshes/holder/cut_rod.obj" scale="0.001 0.001 0.001"/>
             </geometry>
         </collision>

File: ws_ur5e_ballpool/src/moveit_config/config/arm_ur5e.ros2_control.xacro (robot description, xacro)
@@ -1,5 +1,5 @@
 <?xml version="1.0"?>
 <robot xmlns:xacro="http://www.ros.org/wiki/xacro">
-    <xacro:macro name="left_arm_ur5e_ros2_control" params="name initial_positions_file">
+    <xacro:macro name="arm_ur5e_ros2_control" params="name initial_positions_file">
         <xacro:property name="initial_positions" value="${xacro.load_yaml(initial_positions_file)['initial_positions']}"/>
         <ros2_control name="${name}" type="system">
@@ -7,50 +7,50 @@
                 <!-- Qui si ha una lista di plugin: decommentare quello che si vuole usare, e commentare gli altri. -->
                 <!-- PLUGIN PER MUJOCO -->
-                <!-- <plugin>mujoco_ros2_control/MujocoSystemInterface</plugin>
-                <param name="mujoco_model">$(find moveit_config)/config/mujoco_bridge/complete_scene.xml</param> -->
+                <plugin>mujoco_ros2_control/MujocoSystemInterface</plugin>
+                <param name="mujoco_model">$(find moveit_config)/config/mujoco_bridge/complete_scene.xml</param>
                 <!-- PLUGIN PER SOLO RVIZ SIMULATO -->
-                <plugin>mock_components/GenericSystem</plugin>
+                <!-- <plugin>mock_components/GenericSystem</plugin> -->
                 <!-- PLUGIN PER HARDWARE REALE -->
                 <!-- ... TODO -->
             </hardware>
-            <joint name="left_shoulder_pan_joint">
+            <joint name="shoulder_pan_joint">
                 <command_interface name="position"/>
                 <state_interface name="position">
-                  <param name="initial_value">${initial_positions['left_shoulder_pan_joint']}</param>
+                  <param name="initial_value">${initial_positions['shoulder_pan_joint']}</param>
                 </state_interface>
                 <state_interface name="velocity"/>
             </joint>
-            <joint name="left_shoulder_lift_joint">
+            <joint name="shoulder_lift_joint">
                 <command_interface name="position"/>
                 <state_interface name="position">
-                  <param name="initial_value">${initial_positions['left_shoulder_lift_joint']}</param>
+                  <param name="initial_value">${initial_positions['shoulder_lift_joint']}</param>
                 </state_interface>
                 <state_interface name="velocity"/>
             </joint>
-            <joint name="left_elbow_joint">
+            <joint name="elbow_joint">
                 <command_interface name="position"/>
                 <state_interface name="position">
-                  <param name="initial_value">${initial_positions['left_elbow_joint']}</param>
+                  <param name="initial_value">${initial_positions['elbow_joint']}</param>
                 </state_interface>
                 <state_interface name="velocity"/>
             </joint>
-            <joint name="left_wrist_1_joint">
+            <joint name="wrist_1_joint">
                 <command_interface name="position"/>
                 <state_interface name="position">
-                  <param name="initial_value">${initial_positions['left_wrist_1_joint']}</param>
+                  <param name="initial_value">${initial_positions['wrist_1_joint']}</param>
                 </state_interface>
                 <state_interface name="velocity"/>
             </joint>
-            <joint name="left_wrist_2_joint">
+            <joint name="wrist_2_joint">
                 <command_interface name="position"/>
                 <state_interface name="position">
-                  <param name="initial_value">${initial_positions['left_wrist_2_joint']}</param>
+                  <param name="initial_value">${initial_positions['wrist_2_joint']}</param>
                 </state_interface>
                 <state_interface name="velocity"/>
             </joint>
-            <joint name="left_wrist_3_joint">
+            <joint name="wrist_3_joint">
                 <command_interface name="position"/>
                 <state_interface name="position">
-                  <param name="initial_value">${initial_positions['left_wrist_3_joint']}</param>
+                  <param name="initial_value">${initial_positions['wrist_3_joint']}</param>
                 </state_interface>
                 <state_interface name="velocity"/>

Commit message: working on vision node

File: ws_ur5e_ballpool/src/arm_description/urdf/arm.urdf.xacro (robot description, xacro)
@@ -148,3 +148,13 @@
     </joint>
     <!-- NOTA: ANDRÀ TARATO REALISTIACAMENTE CON IL METODO DEL PIVOT!! -->
+    <!-- ========================================== -->
+    <!-- Terna della Telecamera (Parametri Estrinseci) -->
+    <!-- ========================================== -->
+    <link name="camera_color_optical_frame" />
+    <joint name="base_to_camera_joint" type="fixed">
+        <!-- Parent link impostato sulla terna REALE del controller UR -->
+        <parent link="base" />
+        <child link="camera_color_optical_frame" />
+        <origin xyz="-0.288986 -0.473449 0.048187" rpy="0.020224 -0.791766 -1.588972" />
+    </joint>
 </robot>

Commit message: fixing cad, scripts for logging simulated

File: ws_ur5e_ballpool/src/arm_description/urdf/arm.urdf.xacro (robot description, xacro)
@@ -75,5 +75,4 @@
         <origin xyz="-0.188189 0.13575 0.556631" rpy="${3*pi/4} 0 ${-pi/2}" />
     </xacro:ur_robot>
-     <!-- NOTA: ANDRÀ TARATO REALISTIACAMENTE CON IL METODO DEL PIVOT!! -->
     <!-- 1. LINK: HOLDER (CAD) -->
     <link name="holder_link">
@@ -103,5 +102,6 @@
         <parent link="tool0" />
         <child link="holder_link" />
-        <origin xyz="0 0 0" rpy="0 0 0" />
+         <!-- VECCHIO: <origin xyz="0 0 0" rpy="0 0 ${pi/4}" /> -->
+        <origin xyz="0 0 0" rpy="0 0 ${pi/4}" />
     </joint>
     <!-- 2. LINK: CUT ROD -->
@@ -139,13 +139,15 @@
     <!-- ========================================== -->
     <link name="rod_tip_virtual_link" />
-    <!-- FIXED JOINT: CUT ROD -> ROD TIP VIRTUAL -->
-    <joint name="cut_rod_tip_joint" type="fixed">
-        <parent link="cut_rod_link" />
+    <!-- FIXED JOINT DIRETTO: FLANGIA (tool0) -> ROD TIP VIRTUAL -->
+    <joint name="tool0_rod_tip_joint" type="fixed">
+        <!-- posizione del TCP rispetto a tool0 -->
+        <parent link="tool0" />
         <child link="rod_tip_virtual_link" />
-        <!-- Traslazione in metri: x = -120mm, z = 81mm -->
-        <!-- Rotazione: pitch di -90 gradi (-pi/2) per allineare asse Z su asse -X -->
-        <origin xyz="-0.118 0 0.081" rpy="0 ${-pi/2} 0" />
+        <!-- VECCHIO: <origin xyz="-0.118 0 0.081" rpy="0 ${-pi/2} 0" />  -->
+        <origin xyz="-0.115204 -0.108042 0.0825857" rpy="${pi/4} ${-pi/2} 0" />
     </joint>
     <!-- NOTA: ANDRÀ TARATO REALISTIACAMENTE CON IL METODO DEL PIVOT!! -->
+    <!-- NOTA: la terna tool0 in RViz ha l'asse x e l'asse y invertiti rispetto alla terna reale del controller UR5e -->
+    <!-- ecco perché abbiamo cambiato di segno x e y rispetto alla taratura -->
     <!-- ========================================== -->
     <!-- Terna della Telecamera (Parametri Estrinseci) -->

Commit message: fixed bug, restored old cad

File: ws_ur5e_ballpool/src/arm_description/urdf/arm.urdf.xacro (robot description, xacro)
@@ -102,6 +102,6 @@
         <parent link="tool0" />
         <child link="holder_link" />
-         <!-- VECCHIO: <origin xyz="0 0 0" rpy="0 0 ${pi/4}" /> -->
-        <origin xyz="0 0 0" rpy="0 0 ${pi/4}" />
+        <origin xyz="0 0 0" rpy="0 0 0" />
+        <!-- <origin xyz="0 0 0" rpy="0 0 ${pi/4}" /> -->
     </joint>
     <!-- 2. LINK: CUT ROD -->
@@ -144,6 +144,6 @@
         <parent link="tool0" />
         <child link="rod_tip_virtual_link" />
-        <!-- VECCHIO: <origin xyz="-0.118 0 0.081" rpy="0 ${-pi/2} 0" />  -->
-        <origin xyz="-0.115204 -0.108042 0.0825857" rpy="${pi/4} ${-pi/2} 0" />
+        <origin xyz="-0.118 0 0.081" rpy="0 ${-pi/2} 0" />
+        <!-- <origin xyz="-0.115204 -0.108042 0.0825857" rpy="${pi/4} ${-pi/2} 0" /> -->
     </joint>
     <!-- NOTA: ANDRÀ TARATO REALISTIACAMENTE CON IL METODO DEL PIVOT!! -->

Commit message: fixed camera in mujoco

File: ws_ur5e_ballpool/src/arm_description/urdf/arm.urdf.xacro (robot description, xacro)
@@ -150,13 +150,14 @@
     <!-- NOTA: la terna tool0 in RViz ha l'asse x e l'asse y invertiti rispetto alla terna reale del controller UR5e -->
     <!-- ecco perché abbiamo cambiato di segno x e y rispetto alla taratura -->
-    <!-- ========================================== -->
-    <!-- Terna della Telecamera (Parametri Estrinseci) -->
+<!-- ========================================== -->
+    <!-- Terna della Telecamera (MATEMATICAMENTE ESATTA) -->
     <!-- ========================================== -->
     <link name="camera_color_optical_frame" />
     <joint name="base_to_camera_joint" type="fixed">
-        <!-- Parent link impostato sulla terna REALE del controller UR -->
         <parent link="base" />
         <child link="camera_color_optical_frame" />
-        <origin xyz="-0.288986 -0.473449 0.048187" rpy="0.020224 -0.791766 -1.588972" />
+        <!-- X e Y originali, Z corretta aggiungendo l'offset di 16.28 cm -->
+        <!-- RPY originali (che erano già perfetti per puntare in basso al tavolo) -->
+        <origin xyz="-0.288986 -0.473449 0.210840" rpy="0.020224 -0.791766 -1.588972" />
     </joint>
 </robot>

Commit message: corrected tf in vision node

File: ws_ur5e_ballpool/src/arm_description/urdf/arm.urdf.xacro (robot description, xacro)
@@ -150,14 +150,13 @@
     <!-- NOTA: la terna tool0 in RViz ha l'asse x e l'asse y invertiti rispetto alla terna reale del controller UR5e -->
     <!-- ecco perché abbiamo cambiato di segno x e y rispetto alla taratura -->
-<!-- ========================================== -->
-    <!-- Terna della Telecamera (MATEMATICAMENTE ESATTA) -->
+    <!-- ========================================== -->
+    <!-- Terna della Telecamera (Parametri Estrinseci) -->
     <!-- ========================================== -->
     <link name="camera_color_optical_frame" />
     <joint name="base_to_camera_joint" type="fixed">
+        <!-- Parent link impostato sulla terna REALE del controller UR -->
         <parent link="base" />
         <child link="camera_color_optical_frame" />
-        <!-- X e Y originali, Z corretta aggiungendo l'offset di 16.28 cm -->
-        <!-- RPY originali (che erano già perfetti per puntare in basso al tavolo) -->
-        <origin xyz="-0.288986 -0.473449 0.210840" rpy="0.020224 -0.791766 -1.588972" />
+        <origin xyz="-0.288986 -0.473449 0.048187" rpy="0.020224 -0.791766 -1.588972" />
     </joint>
 </robot>

Commit message: Fixed problems for real camera's dept

File: ws_ur5e_ballpool/src/arm_description/urdf/arm.urdf.xacro (robot description, xacro)
@@ -160,3 +160,10 @@
         <origin xyz="-0.288986 -0.473449 0.048187" rpy="0.020224 -0.791766 -1.588972" />
     </joint>
+    <link name="camera_depth_optical_frame" />
+    <joint name="base_to_camera_depth_joint" type="fixed">
+        <!-- Parent link impostato sulla terna REALE del controller UR -->
+        <parent link="base" />
+        <child link="camera_depth_optical_frame" />
+        <origin xyz="-0.288986 -0.473449 0.048187" rpy="0.020224 -0.791766 -1.588972" />
+    </joint>
 </robot>

File: ws_ur5e_ballpool/src/arm_description/urdf/arm_driver_wrapper.urdf.xacro (robot description, xacro)
@@ -62,5 +62,5 @@
             </material>
         </visual>
-        <collision>
+        <collision>terna
             <origin xyz="0 0 0" rpy="0 0 0" />
             <geometry>

Commit message: updated cad

File: ws_ur5e_ballpool/src/arm_description/urdf/arm.urdf.xacro (robot description, xacro)
@@ -102,6 +102,8 @@
         <parent link="tool0" />
         <child link="holder_link" />
+        <!-- vecchio cad -->
+        <!-- <origin xyz="0 0 0" rpy="0 0 0" /> -->
+        <!-- nuovo cad -->
         <origin xyz="0 0 0" rpy="0 0 0" />
-        <!-- <origin xyz="0 0 0" rpy="0 0 ${pi/4}" /> -->
     </joint>
     <!-- 2. LINK: CUT ROD -->
@@ -144,6 +146,8 @@
         <parent link="tool0" />
         <child link="rod_tip_virtual_link" />
-        <origin xyz="-0.118 0 0.081" rpy="0 ${-pi/2} 0" />
-        <!-- <origin xyz="-0.115204 -0.108042 0.0825857" rpy="${pi/4} ${-pi/2} 0" /> -->
+        <!-- vecchio cad -->
+        <!-- <origin xyz="-0.118 0 0.081" rpy="0 ${-pi/2} 0" /> -->
+        <!-- nuovo cad -->
+        <origin xyz="0.115204 0.108042 0.0825857" rpy="${pi/4} ${-pi/2} 0" />
     </joint>
     <!-- NOTA: ANDRÀ TARATO REALISTIACAMENTE CON IL METODO DEL PIVOT!! -->

File: ws_ur5e_ballpool/src/arm_description/urdf/arm_driver_wrapper.urdf.xacro (robot description, xacro)
@@ -62,5 +62,5 @@
             </material>
         </visual>
-        <collision>terna
+        <collision>
             <origin xyz="0 0 0" rpy="0 0 0" />
             <geometry>
@@ -166,4 +166,7 @@
         <parent link="tool0" />
         <child link="holder_link" />
+        <!-- vecchio cad -->
+        <!-- <origin xyz="0 0 0" rpy="0 0 0" /> -->
+        <!-- nuovo cad -->
         <origin xyz="0 0 0" rpy="0 0 0" />
     </joint>
@@ -184,9 +187,9 @@
         <inertial>
             <!-- Centro di massa della Cut Rod in metri -->
-            <origin xyz="-0.029300 0.000000 0.080990" rpy="0 0 0" />
-            <mass value="0.012517" />
-            <inertia ixx="0.0000002222" ixy="0.0000000000" ixz="0.0000000000"
-                     iyy="0.0000262241" iyz="0.0000000000"
-                     izz="0.0000262242" />
+          <origin xyz="-0.029300 0.000000 0.080990" rpy="0 0 0" />
+          <mass value="0.012517" />
+          <inertia ixx="0.0000002222" ixy="0.0000000000" ixz="0.0000000000"
+                   iyy="0.0000262241" iyz="0.0000000000"
+                   izz="0.0000262242" />
         </inertial>
     </link>
@@ -195,4 +198,5 @@
         <parent link="holder_link" />
         <child link="cut_rod_link" />
+        <!-- Se le mesh condividono lo stesso sistema di riferimento zero del CAD, l'origine è 0 0 0 -->
         <origin xyz="0 0 0" rpy="0 0 0" />
     </joint>
@@ -201,11 +205,33 @@
     <!-- ========================================== -->
     <link name="rod_tip_virtual_link" />
-    <!-- FIXED JOINT: CUT ROD -> ROD TIP VIRTUAL -->
-    <joint name="cut_rod_tip_joint" type="fixed">
-        <parent link="cut_rod_link" />
+    <!-- FIXED JOINT DIRETTO: FLANGIA (tool0) -> ROD TIP VIRTUAL -->
+    <joint name="tool0_rod_tip_joint" type="fixed">
+        <!-- posizione del TCP rispetto a tool0 -->
+        <parent link="tool0" />
         <child link="rod_tip_virtual_link" />
-        <!-- Traslazione in metri: x = -120mm, z = 81mm -->
-        <!-- Rotazione: pitch di -90 gradi (-pi/2) per allineare asse Z su asse -X -->
-        <origin xyz="-0.118 0 0.081" rpy="0 ${-pi/2} 0" />
+        <!-- vecchio cad -->
+        <!-- <origin xyz="-0.118 0 0.081" rpy="0 ${-pi/2} 0" /> -->
+        <!-- nuovo cad -->
+        <origin xyz="0.115204 0.108042 0.0825857" rpy="${pi/4} ${-pi/2} 0" />
+    </joint>
+    <!-- NOTA: ANDRÀ TARATO REALISTIACAMENTE CON IL METODO DEL PIVOT!! -->
+    <!-- NOTA: la terna tool0 in RViz ha l'asse x e l'asse y invertiti rispetto alla terna reale del controller UR5e -->
+    <!-- ecco perché abbiamo cambiato di segno x e y rispetto alla taratura -->
+    <!-- ========================================== -->
+    <!-- Terna della Telecamera (Parametri Estrinseci) -->
+    <!-- ========================================== -->
+    <link name="camera_color_optical_frame" />
+    <joint name="base_to_camera_joint" type="fixed">
+        <!-- Parent link impostato sulla terna REALE del controller UR -->
+        <parent link="base" />
+        <child link="camera_color_optical_frame" />
+        <origin xyz="-0.288986 -0.473449 0.048187" rpy="0.020224 -0.791766 -1.588972" />
+    </joint>
+    <link name="camera_depth_optical_frame" />
+    <joint name="base_to_camera_depth_joint" type="fixed">
+        <!-- Parent link impostato sulla terna REALE del controller UR -->
+        <parent link="base" />
+        <child link="camera_depth_optical_frame" />
+        <origin xyz="-0.288986 -0.473449 0.048187" rpy="0.020224 -0.791766 -1.588972" />
     </joint>
 </robot>

File: ws_ur5e_ballpool/src/moveit_config/config/ur5e.ros2_control.xacro (robot description, xacro)
@@ -6,18 +6,18 @@
             <hardware>
                 <!-- PLUGIN PER MUJOCO -->
-                <plugin>mujoco_ros2_control/MujocoSystemInterface</plugin>
-                <param name="mujoco_model">$(find moveit_config)/config/mujoco_bridge/complete_scene.xml</param>
+                <!-- <plugin>mujoco_ros2_control/MujocoSystemInterface</plugin>
+                <param name="mujoco_model">$(find moveit_config)/config/mujoco_bridge/complete_scene.xml</param> -->
                 <!-- PLUGIN PER SOLO RVIZ SIMULATO -->
                 <!-- <plugin>mock_components/GenericSystem</plugin> -->
                 <!-- PLUGIN PER HARDWARE REALE / UrSim -->
-                <!-- <plugin>ur_robot_driver/URPositionHardwareInterface</plugin>
-                <param name="robot_ip">192.168.56.101</param>
+                <plugin>ur_robot_driver/URPositionHardwareInterface</plugin>
+                <param name="robot_ip">192.168.1.110</param>
                 <param name="script_filename">$(find ur_robot_driver)/resources/ros_control.urscript</param>
                 <param name="headless_mode">true</param>
-                <param name="reverse_ip">192.168.56.1</param>
+                <param name="reverse_ip"></param>
                 <param name="reverse_port">50001</param>
                 <param name="script_sender_port">50002</param>
                 <param name="script_command_port">50004</param>
-                <param name="trajectory_port">50003</param> -->
+                <param name="trajectory_port">50003</param>
             </hardware>
             <joint name="shoulder_pan_joint">
