Commit message: fixed cad in arm_description and MuJoCo, add atomic scripts

File: ws_ur5e_ballpool/src/arm_description/urdf/arm.urdf.xacro (robot description, xacro)
@@ -149,9 +149,7 @@
         <!-- <origin xyz="-0.118 0 0.081" rpy="0 ${-pi/2} 0" /> -->
         <!-- nuovo cad -->
-        <origin xyz="0.115204 0.108042 0.0825857" rpy="${pi/4} ${-pi/2} 0" />
+        <origin xyz="0.115204 0.108042 0.0825857" rpy="${radians(43.5 + 180)} ${-pi/2} 0" />
+        <!-- angolo di 43.5° trovato con tuning a mano, per allineare terna TCP con asta (che è curvata) -->
     </joint>
-    <!-- NOTA: ANDRÀ TARATO REALISTIACAMENTE CON IL METODO DEL PIVOT!! -->
-    <!-- NOTA: la terna tool0 in RViz ha l'asse x e l'asse y invertiti rispetto alla terna reale del controller UR5e -->
-    <!-- ecco perché abbiamo cambiato di segno x e y rispetto alla taratura -->
     <!-- ========================================== -->
     <!-- Terna della Telecamera (Parametri Estrinseci) -->

File: ws_ur5e_ballpool/src/arm_description/urdf/arm_driver_wrapper.urdf.xacro (robot description, xacro)
@@ -213,9 +213,8 @@
         <!-- <origin xyz="-0.118 0 0.081" rpy="0 ${-pi/2} 0" /> -->
         <!-- nuovo cad -->
-        <origin xyz="0.115204 0.108042 0.0825857" rpy="${pi/4} ${-pi/2} 0" />
-    </joint>
-    <!-- NOTA: ANDRÀ TARATO REALISTIACAMENTE CON IL METODO DEL PIVOT!! -->
-    <!-- NOTA: la terna tool0 in RViz ha l'asse x e l'asse y invertiti rispetto alla terna reale del controller UR5e -->
-    <!-- ecco perché abbiamo cambiato di segno x e y rispetto alla taratura -->
+        <!-- nuovo cad -->
+        <origin xyz="0.115204 0.108042 0.0825857" rpy="${radians(43.5 + 180)} ${-pi/2} 0" />
+        <!-- angolo di 43.5° trovato con tuning a mano, per allineare terna TCP con asta (che è curvata) -->
+   </joint>
     <!-- ========================================== -->
     <!-- Terna della Telecamera (Parametri Estrinseci) -->

Commit message: something modified

File: ws_ur5e_ballpool/src/arm_description/urdf/arm.urdf.xacro (robot description, xacro)
@@ -155,16 +155,16 @@
     <!-- Terna della Telecamera (Parametri Estrinseci) -->
     <!-- ========================================== -->
-    <link name="camera_color_optical_frame" />
+    <link name="camera_color_frame" />
     <joint name="base_to_camera_joint" type="fixed">
         <!-- Parent link impostato sulla terna REALE del controller UR -->
         <parent link="base" />
-        <child link="camera_color_optical_frame" />
+        <child link="camera_color_frame" />
         <origin xyz="-0.288986 -0.473449 0.048187" rpy="0.020224 -0.791766 -1.588972" />
     </joint>
-    <link name="camera_depth_optical_frame" />
+    <link name="camera_depth_frame" />
     <joint name="base_to_camera_depth_joint" type="fixed">
         <!-- Parent link impostato sulla terna REALE del controller UR -->
         <parent link="base" />
-        <child link="camera_depth_optical_frame" />
+        <child link="camera_depth_frame" />
         <origin xyz="-0.288986 -0.473449 0.048187" rpy="0.020224 -0.791766 -1.588972" />
     </joint>

Commit message: fixing camera tf requirements

File: ws_ur5e_ballpool/src/arm_description/urdf/arm.urdf.xacro (robot description, xacro)
@@ -155,17 +155,25 @@
     <!-- Terna della Telecamera (Parametri Estrinseci) -->
     <!-- ========================================== -->
-    <link name="camera_color_frame" />
-    <joint name="base_to_camera_joint" type="fixed">
-        <!-- Parent link impostato sulla terna REALE del controller UR -->
+    <!-- ========================================== -->
+    <!-- 1. Posizione esatta della Lente RGB (Calibrazione) -->
+    <!-- ========================================== -->
+    <link name="camera_rgb_calibrated" />
+    <joint name="base_to_rgb_joint" type="fixed">
         <parent link="base" />
-        <child link="camera_color_frame" />
+        <child link="camera_rgb_calibrated" />
         <origin xyz="-0.288986 -0.473449 0.048187" rpy="0.020224 -0.791766 -1.588972" />
     </joint>
-    <link name="camera_depth_frame" />
-    <joint name="base_to_camera_depth_joint" type="fixed">
-        <!-- Parent link impostato sulla terna REALE del controller UR -->
-        <parent link="base" />
-        <child link="camera_depth_frame" />
-        <origin xyz="-0.288986 -0.473449 0.048187" rpy="0.020224 -0.791766 -1.588972" />
+    <!-- ========================================== -->
+    <!-- 2. Offset fisico su +X (1.48cm) + Rotazione asse Z -->
+    <!-- ========================================== -->
+    <link name="camera_link" />
+    <joint name="rgb_to_camera_link_joint" type="fixed">
+        <parent link="camera_rgb_calibrated" />
+        <child link="camera_link" />
+        <!--
+          Traslazione (xyz): Sposta di 1.48 cm lungo l'asse X positivo (0.0148).
+          Rotazione (rpy): Ruota di 90 gradi (1.5708 rad) su Z.
+        -->
+        <origin xyz="0.0148 0 0" rpy="0 0 1.5708" />
     </joint>
 </robot>

Commit message: fixed Calibration

File: ws_ur5e_ballpool/src/arm_description/urdf/arm.urdf.xacro (robot description, xacro)
@@ -162,5 +162,5 @@
         <parent link="base" />
         <child link="camera_rgb_calibrated" />
-        <origin xyz="-0.288986 -0.473449 0.048187" rpy="0.020224 -0.791766 -1.588972" />
+        <origin xyz="-0.28898614560797165 -0.4734488805016898 0.04818685648725712" rpy="0.02022358 -0.79176606 -1.58897229" />
     </joint>
     <!-- ========================================== -->
@@ -175,5 +175,5 @@
           Rotazione (rpy): Ruota di 90 gradi (1.5708 rad) su Z.
         -->
-        <origin xyz="0.0148 0 0" rpy="0 0 1.5708" />
+         <origin xyz="0.0178 -0.0088 0.0266" rpy="0 -1.5708 1.5708" />
     </joint>
 </robot>

File: ws_ur5e_ballpool/src/arm_description/urdf/arm_driver_wrapper.urdf.xacro (robot description, xacro)
@@ -220,17 +220,29 @@
     <!-- Terna della Telecamera (Parametri Estrinseci) -->
     <!-- ========================================== -->
-    <link name="camera_color_optical_frame" />
-    <joint name="base_to_camera_joint" type="fixed">
-        <!-- Parent link impostato sulla terna REALE del controller UR -->
+    <!-- ========================================== -->
+    <!-- 1. Posizione esatta della Lente RGB (Calibrazione) -->
+    <!-- ========================================== -->
+    <link name="camera_rgb_calibrated" />
+    <joint name="base_to_rgb_joint" type="fixed">
         <parent link="base" />
-        <child link="camera_color_optical_frame" />
-        <origin xyz="-0.288986 -0.473449 0.048187" rpy="0.020224 -0.791766 -1.588972" />
-    </joint>
-    <link name="camera_depth_optical_frame" />
-    <joint name="base_to_camera_depth_joint" type="fixed">
-        <!-- Parent link impostato sulla terna REALE del controller UR -->
-        <parent link="base" />
-        <child link="camera_depth_optical_frame" />
-        <origin xyz="-0.288986 -0.473449 0.048187" rpy="0.020224 -0.791766 -1.588972" />
+        <child link="camera_rgb_calibrated" />
+        <origin xyz="-0.28898614560797165 -0.4734488805016898 0.04818685648725712" rpy="0.02022358 -0.79176606 -1.58897229" />
+    </joint>
+    <!-- ========================================== -->
+    <!-- 2. Offset fisico su +X (1.48cm) + Rotazione asse Z -->
+    <!-- ========================================== -->
+    <link name="camera_link" />
+    <joint name="rgb_to_camera_link_joint" type="fixed">
+        <parent link="camera_rgb_calibrated" />
+        <child link="camera_link" />
+        <!--
+          Traslazione (xyz): Sposta di 1.48 cm lungo l'asse X positivo (0.0148).
+          Rotazione (rpy): Ruota di 90 gradi (1.5708 rad) su Z.
+        -->
+        <!-- <origin xyz="0.0148 0.0 0.00" rpy="0 -1.5708 1.5708" /> -->
+        <!-- <origin xyz="0.0178 -0.0088 0.0286" rpy="0 -1.5708 1.5708" /> -->
+        <!-- <origin xyz="0.0130 -0.0080 0.0287" rpy="0 -1.5708 1.5708" /> -->
+        <!-- <origin xyz="0.0133 -0.0080 0.0287" rpy="0 -1.5708 1.6232" /> -->
+        <origin xyz="0.0130 -0.0120 0.0287" rpy="0 -1.5708 1.5883" />
     </joint>
 </robot>

Commit message: added test_tip_positioning in simulation

File: ws_ur5e_ballpool/src/arm_description/urdf/arm.urdf.xacro (robot description, xacro)
@@ -152,28 +152,14 @@
         <!-- angolo di 43.5° trovato con tuning a mano, per allineare terna TCP con asta (che è curvata) -->
     </joint>
-    <!-- ========================================== -->
+    <!-- ====================================================== -->
     <!-- Terna della Telecamera (Parametri Estrinseci) -->
-    <!-- ========================================== -->
-    <!-- ========================================== -->
-    <!-- 1. Posizione esatta della Lente RGB (Calibrazione) -->
-    <!-- ========================================== -->
-    <link name="camera_rgb_calibrated" />
-    <joint name="base_to_rgb_joint" type="fixed">
+    <!-- ====================================================== -->
+    <link name="camera_color_optical_frame" />
+    <joint name="base_to_camera_joint" type="fixed">
+        <!-- Parent link imposto sulla terna REALE del controller UR -->
         <parent link="base" />
-        <child link="camera_rgb_calibrated" />
-        <origin xyz="-0.28898614560797165 -0.4734488805016898 0.04818685648725712" rpy="0.02022358 -0.79176606 -1.58897229" />
-    </joint>
-    <!-- ========================================== -->
-    <!-- 2. Offset fisico su +X (1.48cm) + Rotazione asse Z -->
-    <!-- ========================================== -->
-    <link name="camera_link" />
-    <joint name="rgb_to_camera_link_joint" type="fixed">
-        <parent link="camera_rgb_calibrated" />
-        <child link="camera_link" />
-        <!--
-          Traslazione (xyz): Sposta di 1.48 cm lungo l'asse X positivo (0.0148).
-          Rotazione (rpy): Ruota di 90 gradi (1.5708 rad) su Z.
-        -->
-         <origin xyz="0.0178 -0.0088 0.0266" rpy="0 -1.5708 1.5708" />
+        <child link="camera_color_optical_frame" />
+        <!-- Parametri estrinseci della telecamera RGB (dalla calibrazione)-->
+        <origin xyz="-0.288986 -0.473449 0.048187" rpy="0.020224 -0.791766 -1.588972" />
     </joint>
 </robot>

File: ws_ur5e_ballpool/src/arm_description/urdf/arm_driver_wrapper.urdf.xacro (robot description, xacro)
@@ -218,9 +218,7 @@
    </joint>
     <!-- ========================================== -->
-    <!-- Terna della Telecamera (Parametri Estrinseci) -->
-    <!-- ========================================== -->
-    <!-- ========================================== -->
-    <!-- 1. Posizione esatta della Lente RGB (Calibrazione) -->
-    <!-- ========================================== -->
+    <!-- Terna della Telecamera -->
+    <!-- ========================================== -->
+    <!-- Posizione della lente RGB rispetto alla base ricavata dalla calibrazione -->
     <link name="camera_rgb_calibrated" />
     <joint name="base_to_rgb_joint" type="fixed">
@@ -229,16 +227,15 @@
         <origin xyz="-0.28898614560797165 -0.4734488805016898 0.04818685648725712" rpy="0.02022358 -0.79176606 -1.58897229" />
     </joint>
-    <!-- ========================================== -->
-    <!-- 2. Offset fisico su +X (1.48cm) + Rotazione asse Z -->
-    <!-- ========================================== -->
+    <!-- Posizione della telecamera (per definizione nel sensore di Depth) rispetto alla lente RGB -->
+    <!-- La lente di depth è traslata di 1.48 cm lungo x rispetto all'RGB -->
+    <!-- riferimenti: https://github.com/realsenseai/realsense-ros/tree/ros2-master -->
+    <!-- Tuttavia, sono inseriti qui anche rotazioni e traslazioni di una calibrazione a mano, per correggere l'allineamento -->
     <link name="camera_link" />
     <joint name="rgb_to_camera_link_joint" type="fixed">
         <parent link="camera_rgb_calibrated" />
         <child link="camera_link" />
-        <!--
-          Traslazione (xyz): Sposta di 1.48 cm lungo l'asse X positivo (0.0148).
-          Rotazione (rpy): Ruota di 90 gradi (1.5708 rad) su Z.
-        -->
+        <!-- SENZA CALIBRAZIONE (solo traslazione lungo x per depth da costruzione del sensore) -->
         <!-- <origin xyz="0.0148 0.0 0.00" rpy="0 -1.5708 1.5708" /> -->
+        <!-- TENTATIVI DI CALIBRAZIONE A MANO -->
         <!-- <origin xyz="0.0178 -0.0088 0.0286" rpy="0 -1.5708 1.5708" /> -->
         <!-- <origin xyz="0.0130 -0.0080 0.0287" rpy="0 -1.5708 1.5708" /> -->

File: ws_ur5e_ballpool/src/moveit_config/config/ur5e.ros2_control.xacro (robot description, xacro)
@@ -9,15 +9,15 @@
                 <param name="mujoco_model">$(find moveit_config)/config/mujoco_bridge/complete_scene.xml</param> -->
                 <!-- PLUGIN PER SOLO RVIZ SIMULATO -->
-                <!-- <plugin>mock_components/GenericSystem</plugin> -->
+                <plugin>mock_components/GenericSystem</plugin>
                 <!-- PLUGIN PER HARDWARE REALE / UrSim -->
-                <plugin>ur_robot_driver/URPositionHardwareInterface</plugin>
-                <param name="robot_ip">192.168.1.110</param>
+                <!-- <plugin>ur_robot_driver/URPositionHardwareInterface</plugin>
+                <param name="robot_ip">192.168.56.101</param>
                 <param name="script_filename">$(find ur_robot_driver)/resources/ros_control.urscript</param>
                 <param name="headless_mode">true</param>
-                <param name="reverse_ip"></param>
+                <param name="reverse_ip">192.168.56.1</param>
                 <param name="reverse_port">50001</param>
                 <param name="script_sender_port">50002</param>
                 <param name="script_command_port">50004</param>
-                <param name="trajectory_port">50003</param>
+                <param name="trajectory_port">50003</param> -->
             </hardware>
             <joint name="shoulder_pan_joint">
