Commit message: trying to fix Ur driver (not working yet)

File: ws_ur5e_ballpool/src/arm_description/urdf/arm_driver_wrapper.urdf.xacro (robot description, xacro)
@@ -1,22 +1,54 @@
 <?xml version="1.0"?>
 <robot name="ur5e" xmlns:xacro="http://ros.org/wiki/xacro">
-    <!-- robot name parameter -->
+    <!-- ========================================== -->
+    <!-- 1. PARAMETRI DI INPUT (Fisica e Hardware)  -->
+    <!-- ========================================== -->
     <xacro:arg name="name" default="ur5e"/>
-     <!-- import main macro dell'UR (richiede pacchetto scaricato Universal Robots -> ur_description) -->
-    <xacro:include filename="$(find ur_description)/urdf/ur_macro.xacro"/>
-    <!-- ROBOT XACRO PARAMETERS-->
     <xacro:arg name="ur_type" default="ur5e"/>
-    <!-- LETTURA PARAMETRI DELL'UR5e DA CONFIG FILES -->
-    <!-- da ur_description, pacchetto ROS (generici UR5e)-->
+    <xacro:arg name="tf_prefix" default=""/>
+    <!-- Parametri UR -->
     <xacro:arg name="joint_limit_params" default="$(find ur_description)/config/$(arg ur_type)/joint_limits.yaml"/>
     <xacro:arg name="physical_params" default="$(find ur_description)/config/$(arg ur_type)/physical_parameters.yaml"/>
     <xacro:arg name="visual_params" default="$(find ur_description)/config/$(arg ur_type)/visual_parameters.yaml"/>
-    <!-- da calibrazione su nostro braccio -->
+    <!-- Da calibrazione su nostro braccio -->
     <xacro:arg name="kinematics_params" default="$(find arm_description)/config/uclv_right_ur5e_kinematics.yaml"/>
-    <!-- safety parameters (ininfluenti in visualizzazione)-->
+    <!-- Parametri Sicurezza -->
     <xacro:arg name="safety_limits" default="true"/>
     <xacro:arg name="safety_pos_margin" default="0.15"/>
     <xacro:arg name="safety_k_position" default="20"/>
-    <!-- DESCRIZIONE STRUTTURALE-->
+    <!-- Parametri Hardware Control (Aggiunti per il driver reale) -->
+    <xacro:arg name="robot_ip" default="0.0.0.0" />
+    <xacro:arg name="headless_mode" default="false" />
+    <xacro:arg name="script_filename" default=""/>
+    <xacro:arg name="output_recipe_filename" default=""/>
+    <xacro:arg name="input_recipe_filename" default=""/>
+    <xacro:arg name="reverse_ip" default="0.0.0.0"/>
+    <xacro:arg name="script_command_port" default="50004"/>
+    <xacro:arg name="reverse_port" default="50001"/>
+    <xacro:arg name="script_sender_port" default="50002"/>
+    <xacro:arg name="trajectory_port" default="50003"/>
+    <xacro:arg name="use_tool_communication" default="false" />
+    <xacro:arg name="tool_voltage" default="0" />
+    <xacro:arg name="tool_parity" default="0" />
+    <xacro:arg name="tool_baud_rate" default="115200" />
+    <xacro:arg name="tool_stop_bits" default="1" />
+    <xacro:arg name="tool_rx_idle_chars" default="1.5" />
+    <xacro:arg name="tool_tx_idle_chars" default="3.5" />
+    <xacro:arg name="tool_device_name" default="/tmp/ttyUR" />
+    <xacro:arg name="tool_tcp_port" default="54321" />
+    <xacro:arg name="use_mock_hardware" default="false" />
+    <xacro:arg name="mock_sensor_commands" default="false" />
+    <xacro:arg name="sim_gazebo" default="false" />
+    <xacro:arg name="sim_ignition" default="false" />
+    <xacro:arg name="simulation_controllers" default="" />
+    <xacro:arg name="initial_positions_file" default="$(find ur_description)/config/initial_positions.yaml"/>
+    <!-- ========================================== -->
+    <!-- 2. IMPORT DELLE MACRO UNIVERSAL ROBOTS     -->
+    <!-- ========================================== -->
+    <xacro:include filename="$(find ur_description)/urdf/ur_macro.xacro"/>
+    <xacro:include filename="$(find ur_robot_driver)/urdf/ur.ros2_control.xacro"/>
+    <!-- ========================================== -->
+    <!-- 3. DESCRIZIONE STRUTTURALE AMBIENTE        -->
+    <!-- ========================================== -->
     <!-- table as base for the UR5e robot -->
     <link name="world">
@@ -60,4 +92,7 @@
         <origin xyz="0 0 0" rpy="0 0 0" />
     </joint>
+    <!-- ========================================== -->
+    <!-- 4. ISTANZIAZIONE ROBOT E HARDWARE INTERFACE-->
+    <!-- ========================================== -->
     <!-- arm -->
     <xacro:ur_robot
@@ -75,4 +110,33 @@
         <origin xyz="-0.188189 0.13575 0.556631" rpy="${3*pi/4} 0 ${-pi/2}" />
     </xacro:ur_robot>
+    <!-- hardware interface per connettersi a URSim o robot reale -->
+    <xacro:ur_ros2_control
+        name="$(arg name)"
+        tf_prefix="$(arg tf_prefix)"
+        kinematics_parameters_file="$(arg kinematics_params)"
+        robot_ip="$(arg robot_ip)"
+        script_filename="$(arg script_filename)"
+        output_recipe_filename="$(arg output_recipe_filename)"
+        input_recipe_filename="$(arg input_recipe_filename)"
+        reverse_ip="$(arg reverse_ip)"
+        script_command_port="$(arg script_command_port)"
+        reverse_port="$(arg reverse_port)"
+        script_sender_port="$(arg script_sender_port)"
+        trajectory_port="$(arg trajectory_port)"
+        use_tool_communication="$(arg use_tool_communication)"
+        tool_voltage="$(arg tool_voltage)"
+        tool_parity="$(arg tool_parity)"
+        tool_baud_rate="$(arg tool_baud_rate)"
+        tool_stop_bits="$(arg tool_stop_bits)"
+        tool_rx_idle_chars="$(arg tool_rx_idle_chars)"
+        tool_tx_idle_chars="$(arg tool_tx_idle_chars)"
+        tool_device_name="$(arg tool_device_name)"
+        tool_tcp_port="$(arg tool_tcp_port)"
+        use_mock_hardware="$(arg use_mock_hardware)"
+        mock_sensor_commands="$(arg mock_sensor_commands)"
+        headless_mode="$(arg headless_mode)"/>
+    <!-- ========================================== -->
+    <!-- 5. END EFFECTOR E STRUMENTI               -->
+    <!-- ========================================== -->
     <!-- 1. LINK: HOLDER (CAD) -->
     <link name="holder_link">
@@ -120,9 +184,9 @@
         <inertial>
             <!-- Centro di massa della Cut Rod in metri -->
-          <origin xyz="-0.029300 0.000000 0.080990" rpy="0 0 0" />
-          <mass value="0.012517" />
-          <inertia ixx="0.0000002222" ixy="0.0000000000" ixz="0.0000000000"
-                   iyy="0.0000262241" iyz="0.0000000000"
-                   izz="0.0000262242" />
+            <origin xyz="-0.029300 0.000000 0.080990" rpy="0 0 0" />
+            <mass value="0.012517" />
+            <inertia ixx="0.0000002222" ixy="0.0000000000" ixz="0.0000000000"
+                     iyy="0.0000262241" iyz="0.0000000000"
+                     izz="0.0000262242" />
         </inertial>
     </link>
@@ -131,5 +195,4 @@
         <parent link="holder_link" />
         <child link="cut_rod_link" />
-        <!-- Se le mesh condividono lo stesso sistema di riferimento zero del CAD, l'origine è 0 0 0 -->
         <origin xyz="0 0 0" rpy="0 0 0" />
     </joint>
@@ -146,4 +209,3 @@
         <origin xyz="-0.118 0 0.081" rpy="0 ${-pi/2} 0" />
     </joint>
-    <!-- NOTA: ANDRÀ TARATO REALISTIACAMENTE CON IL METODO DEL PIVOT!! -->
 </robot>

File: ws_ur5e_ballpool/src/moveit_config/config/ur5e.ros2_control.xacro (robot description, xacro)
@@ -1,5 +1,5 @@
 <?xml version="1.0"?>
 <robot xmlns:xacro="http://www.ros.org/wiki/xacro">
-    <xacro:macro name="arm_ur5e_ros2_control" params="name initial_positions_file">
+    <xacro:macro name="ur5e_ros2_control" params="name initial_positions_file">
         <xacro:property name="initial_positions" value="${xacro.load_yaml(initial_positions_file)['initial_positions']}"/>
         <ros2_control name="${name}" type="system">
@@ -10,10 +10,16 @@
                 <param name="mujoco_model">$(find moveit_config)/config/mujoco_bridge/complete_scene.xml</param> -->
                 <!-- PLUGIN PER SOLO RVIZ SIMULATO -->
-                <plugin>mock_components/GenericSystem</plugin>
-                <!-- PLUGIN PER HARDWARE REALE -->
-                <!-- ... TODO -->
+                <!-- <plugin>mock_components/GenericSystem</plugin> -->
+                <!-- PLUGIN PER HARDWARE REALE / UrSim -->
+                <plugin>ur_robot_driver/URPositionHardwareInterface</plugin>
+                <param name="robot_ip">192.168.56.101</param>
+                <param name="script_filename">$(find ur_robot_driver)/resources/ros_cocontrol.urscript</param>
+                <param name="headless_mode">true</param>
+                <param name="reverse_port">50001</param>
+                <param name="script_sender_port">50002</param>
             </hardware>
             <joint name="shoulder_pan_joint">
                 <command_interface name="position"/>
+                <command_interface name="velocity"/>
                 <state_interface name="position">
                   <param name="initial_value">${initial_positions['shoulder_pan_joint']}</param>
@@ -23,4 +29,5 @@
             <joint name="shoulder_lift_joint">
                 <command_interface name="position"/>
+                <command_interface name="velocity"/>
                 <state_interface name="position">
                   <param name="initial_value">${initial_positions['shoulder_lift_joint']}</param>
@@ -30,4 +37,5 @@
             <joint name="elbow_joint">
                 <command_interface name="position"/>
+                <command_interface name="velocity"/>
                 <state_interface name="position">
                   <param name="initial_value">${initial_positions['elbow_joint']}</param>
@@ -37,4 +45,5 @@
             <joint name="wrist_1_joint">
                 <command_interface name="position"/>
+                <command_interface name="velocity"/>
                 <state_interface name="position">
                   <param name="initial_value">${initial_positions['wrist_1_joint']}</param>
@@ -44,4 +53,5 @@
             <joint name="wrist_2_joint">
                 <command_interface name="position"/>
+                <command_interface name="velocity"/>
                 <state_interface name="position">
                   <param name="initial_value">${initial_positions['wrist_2_joint']}</param>
@@ -51,4 +61,5 @@
             <joint name="wrist_3_joint">
                 <command_interface name="position"/>
+                <command_interface name="velocity"/>
                 <state_interface name="position">
                   <param name="initial_value">${initial_positions['wrist_3_joint']}</param>

Commit message: removed compressed

File: ws_ur5e_ballpool/src/arm_description/urdf/arm_driver_wrapper.urdf.xacro (robot description, xacro)
@@ -241,5 +241,7 @@
         <!-- <origin xyz="0.0130 -0.0080 0.0287" rpy="0 -1.5708 1.5708" /> -->
         <!-- <origin xyz="0.0133 -0.0080 0.0287" rpy="0 -1.5708 1.6232" /> -->
-        <origin xyz="0.0130 -0.0120 0.0287" rpy="0 -1.5708 1.5883" />
+        <!-- <origin xyz="0.0130 -0.0120 0.0287" rpy="0 -1.5708 1.5883" />  -->
+        <!-- <origin xyz="0.0130 -0.0020 0.0280" rpy="0 -1.5708 1.5883" />  -->
+        <origin xyz="0.0130 -0.0020 0.0350" rpy="0 -1.5708 1.5920" />
     </joint>
 </robot>

Commit message: calibration camera AGAIN

File: ws_ur5e_ballpool/src/arm_description/urdf/arm_driver_wrapper.urdf.xacro (robot description, xacro)
@@ -241,7 +241,10 @@
         <!-- <origin xyz="0.0130 -0.0080 0.0287" rpy="0 -1.5708 1.5708" /> -->
         <!-- <origin xyz="0.0133 -0.0080 0.0287" rpy="0 -1.5708 1.6232" /> -->
+        <!-- PRIMA DI OGGI -->
         <!-- <origin xyz="0.0130 -0.0120 0.0287" rpy="0 -1.5708 1.5883" />  -->
+        <!-- OGGI -->
         <!-- <origin xyz="0.0130 -0.0020 0.0280" rpy="0 -1.5708 1.5883" />  -->
-        <origin xyz="0.0130 -0.0020 0.0350" rpy="0 -1.5708 1.5920" />
+        <origin xyz="0.018 -0.004 0.031" rpy="0 -1.5708 1.5883" />
+        <!-- <origin xyz="0.018 -0.004 0.031" rpy="0 -1.5708 1.5935" />  -->
     </joint>
 </robot>

Commit message: final push with analysis

File: ws_ur5e_ballpool/src/arm_description/urdf/arm_driver_wrapper.urdf.xacro (robot description, xacro)
@@ -241,10 +241,11 @@
         <!-- <origin xyz="0.0130 -0.0080 0.0287" rpy="0 -1.5708 1.5708" /> -->
         <!-- <origin xyz="0.0133 -0.0080 0.0287" rpy="0 -1.5708 1.6232" /> -->
-        <!-- PRIMA DI OGGI -->
         <!-- <origin xyz="0.0130 -0.0120 0.0287" rpy="0 -1.5708 1.5883" />  -->
-        <!-- OGGI -->
         <!-- <origin xyz="0.0130 -0.0020 0.0280" rpy="0 -1.5708 1.5883" />  -->
+        <!-- LAST VALID (30-09) -->
         <origin xyz="0.018 -0.004 0.031" rpy="0 -1.5708 1.5883" />
-        <!-- <origin xyz="0.018 -0.004 0.031" rpy="0 -1.5708 1.5935" />  -->
+        <!-- OCTOBER 05 -->
+        <!-- <origin xyz="0.018 -0.004 0.031" rpy="0 -1.5708 1.5970" />  -->
+        <!-- <origin xyz="0.018 -0.004 0.031" rpy="0 -1.5708 1.6057" />  -->
     </joint>
 </robot>
